Commit message: Trying to import the controller

File: 41068_ws/src/41068_ignition_bringup/urdf/Quadruped_URDF/robot.xacro (robot description, xacro)
@@ -1,5 +1,8 @@
 <?xml version="1.0"?>
 <robot name="acs_robot" xmlns:xacro="http://ros.org/wiki/xacro">
-  <!-- Parts -->
+  <!-- ================== Args ================== -->
+  <!-- Path to controller config YAML, passed from launch -->
+  <xacro:arg name="controller_config" default="$(find 41068_ignition_bringup)/config/robot_controller.yaml"/>
+  <!-- ================== Includes ================== -->
   <xacro:include filename="$(find 41068_ignition_bringup)/urdf/Quadruped_URDF/base.xacro"/>
   <xacro:include filename="$(find 41068_ignition_bringup)/urdf/Quadruped_URDF/leg_joint.xacro"/>
@@ -10,5 +13,5 @@
   <xacro:include filename="$(find 41068_ignition_bringup)/urdf/Quadruped_URDF/robot_control_gazebo.xacro"/>
   <xacro:property name="PI" value="3.14159274"/>
-  <!-- =============== Link & Joint =============== -->
+  <!-- ================== Links & Joints ================== -->
   <!-- Base -->
   <link name="base_footprint"/>
@@ -16,7 +19,8 @@
     <origin xyz="0 0 0" rpy="0 0 0" />
   </xacro:base>
+  <!-- Leg joints -->
   <xacro:leg_joint_v0 prefix="rear_left" parent="base_link">
     <origin xyz="-0.277 0.06 0.089405" rpy="0 ${PI/2} ${-PI/2}"/>
-    <axis xyz="0 -1 0"/> <!-- 0 -1 0 -->
+    <axis xyz="0 -1 0"/>
   </xacro:leg_joint_v0>
   <xacro:leg_joint_v0 prefix="rear_right" parent="base_link">
@@ -26,5 +30,5 @@
   <xacro:leg_joint_v0 prefix="front_left" parent="base_link">
     <origin xyz="0.282 0.06 0.090255" rpy="0 ${PI/2} ${-PI/2}"/>
-    <axis xyz="0 -1 0"/> <!-- 0 -1 0 -->
+    <axis xyz="0 -1 0"/>
   </xacro:leg_joint_v0>
   <xacro:leg_joint_v0 prefix="front_right" parent="base_link">
@@ -32,4 +36,5 @@
     <axis xyz="0 1 0"/>
   </xacro:leg_joint_v0>
+  <!-- Thighs -->
   <xacro:left_thigh_v0 prefix="front" parent="front_left_leg_joint_link">
     <origin xyz="0 0 -0.114" rpy="${PI/2} 0 ${-PI/2}"/>
@@ -42,10 +47,11 @@
   <xacro:right_thigh_v0 prefix="front" parent="front_right_leg_joint_link">
     <origin xyz="0 0 -0.114" rpy="${PI/2} 0 ${-PI/2}"/>
-    <axis xyz="0 -1 0"/> <!-- 0 -1 0 -->
+    <axis xyz="0 -1 0"/>
   </xacro:right_thigh_v0>
   <xacro:right_thigh_v0 prefix="rear" parent="rear_right_leg_joint_link">
     <origin xyz="0 0 -0.114" rpy="${PI/2} 0 ${-PI/2}"/>
-    <axis xyz="0 -1 0"/> <!-- 0 -1 0 -->
+    <axis xyz="0 -1 0"/>
   </xacro:right_thigh_v0>
+  <!-- Shins -->
   <xacro:shin_v0 prefix="front_left" parent="front_left_thigh_link">
     <origin xyz="0.426 -0.0285 0" rpy="0 0 0"/>
@@ -64,8 +70,8 @@
     <axis xyz="0 1 0"/>
   </xacro:shin_v0>
-  <!-- =============== Gazebo =============== -->
+  <!-- ================== Gazebo Plugins ================== -->
   <!-- Controllers -->
-  <xacro:robot_ros2_control/>
-  <!-- Base -->
+  <xacro:robot_ros2_control controller_config="$(arg controller_config)"/>
+  <!-- Visual/Gazebo tags for parts -->
   <xacro:base_gazebo_v0/>
   <xacro:leg_joint_gazebo_v0 prefix="rear_left"/>

File: 41068_ws/src/41068_ignition_bringup/urdf/Quadruped_URDF/robot_control_gazebo.xacro (robot description, xacro)
@@ -1,85 +1,79 @@
 <?xml version="1.0" ?>
 <robot xmlns:xacro="http://www.ros.org/wiki/xacro">
-<xacro:macro name="robot_ros2_control">
-  <!-- ros2_control block -->
-  <ros2_control name="gazebo_system" type="system">
-    <hardware>
-      <plugin>gz_ros2_control/GazeboSimSystem</plugin>
-    </hardware>
-    <!-- All joints -->
-    <joint name="front_left_leg_joint">
-      <command_interface name="position"/>
-      <state_interface name="position"/>
-    </joint>
-    <joint name="front_right_leg_joint">
-      <command_interface name="position"/>
-      <state_interface name="position"/>
-    </joint>
-    <joint name="rear_left_leg_joint">
-      <command_interface name="position"/>
-      <state_interface name="position"/>
-    </joint>
-    <joint name="rear_right_leg_joint">
-      <command_interface name="position"/>
-      <state_interface name="position"/>
-    </joint>
-    <joint name="front_left_thigh_joint">
-      <command_interface name="position"/>
-      <state_interface name="position"/>
-    </joint>
-    <joint name="front_right_thigh_joint">
-      <command_interface name="position"/>
-      <state_interface name="position"/>
-    </joint>
-    <joint name="rear_left_thigh_joint">
-      <command_interface name="position"/>
-      <state_interface name="position"/>
-    </joint>
-    <joint name="rear_right_thigh_joint">
-      <command_interface name="position"/>
-      <state_interface name="position"/>
-    </joint>
-    <joint name="front_left_shin_joint">
-      <command_interface name="position"/>
-      <state_interface name="position"/>
-    </joint>
-    <joint name="front_right_shin_joint">
-      <command_interface name="position"/>
-      <state_interface name="position"/>
-    </joint>
-    <joint name="rear_left_shin_joint">
-      <command_interface name="position"/>
-      <state_interface name="position"/>
-    </joint>
-    <joint name="rear_right_shin_joint">
-      <command_interface name="position"/>
-      <state_interface name="position"/>
-    </joint>
-  </ros2_control>
-  <!-- Gazebo plugins -->
-  <gazebo>
-    <plugin
-      filename="gz_ros2_control-system"
-      name="gz_ros2_control::GazeboSimROS2ControlPlugin">
-      <ros2_parameters>
-        <use_sim_time>true</use_sim_time>
-        <robot_description>/quadruped/robot_description</robot_description>
-        <parameters>$(find 41068_ignition_bringup)/config/robot_controller.yaml</parameters>
-      </ros2_parameters>
-    </plugin>
-    <plugin
-      filename="libgz-sim-joint-state-publisher-system"
-      name="gz::sim::systems::JointStatePublisher"/>
-    <plugin
-      filename="libgz-sim-pose-publisher-system"
-      name="gz::sim::systems::PosePublisher">
-      <publish_link_pose>true</publish_link_pose>
-      <use_pose_vector_msg>true</use_pose_vector_msg>
-      <publish_nested_model_pose>true</publish_nested_model_pose>
-    </plugin>
-    <plugin
-      filename="gz-sim-imu-system"
-      name="gz::sim::systems::Imu"/>
-  </gazebo>
-</xacro:macro>
+  <xacro:macro name="robot_ros2_control" params="controller_config">
+    <!-- ros2_control block -->
+    <ros2_control name="gazebo_system" type="system">
+      <hardware>
+        <plugin>gz_ros2_control/GazeboSimSystem</plugin>
+      </hardware>
+      <!-- All joints -->
+      <joint name="front_left_leg_joint">
+        <command_interface name="position"/>
+        <state_interface name="position"/>
+      </joint>
+      <joint name="front_right_leg_joint">
+        <command_interface name="position"/>
+        <state_interface name="position"/>
+      </joint>
+      <joint name="rear_left_leg_joint">
+        <command_interface name="position"/>
+        <state_interface name="position"/>
+      </joint>
+      <joint name="rear_right_leg_joint">
+        <command_interface name="position"/>
+        <state_interface name="position"/>
+      </joint>
+      <joint name="front_left_thigh_joint">
+        <command_interface name="position"/>
+        <state_interface name="position"/>
+      </joint>
+      <joint name="front_right_thigh_joint">
+        <command_interface name="position"/>
+        <state_interface name="position"/>
+      </joint>
+      <joint name="rear_left_thigh_joint">
+        <command_interface name="position"/>
+        <state_interface name="position"/>
+      </joint>
+      <joint name="rear_right_thigh_joint">
+        <command_interface name="position"/>
+        <state_interface name="position"/>
+      </joint>
+      <joint name="front_left_shin_joint">
+        <command_interface name="position"/>
+        <state_interface name="position"/>
+      </joint>
+      <joint name="front_right_shin_joint">
+        <command_interface name="position"/>
+        <state_interface name="position"/>
+      </joint>
+      <joint name="rear_left_shin_joint">
+        <command_interface name="position"/>
+        <state_interface name="position"/>
+      </joint>
+      <joint name="rear_right_shin_joint">
+        <command_interface name="position"/>
+        <state_interface name="position"/>
+      </joint>
+    </ros2_control>
+    <!-- Gazebo plugin -->
+    <gazebo>
+      <plugin
+        filename="gz_ros2_control-system"
+        name="gz_ros2_control::GazeboSimROS2ControlPlugin">
+        <ros2_parameters>
+          <ros2_parameter_file>${controller_config}</ros2_parameter_file>
+        </ros2_parameters>
+      </plugin>
+      <plugin filename="libgz-sim-joint-state-publisher-system"
+              name="gz::sim::systems::JointStatePublisher"/>
+      <plugin filename="libgz-sim-pose-publisher-system"
+              name="gz::sim::systems::PosePublisher">
+        <publish_link_pose>true</publish_link_pose>
+        <use_pose_vector_msg>true</use_pose_vector_msg>
+        <publish_nested_model_pose>true</publish_nested_model_pose>
+      </plugin>
+      <plugin filename="gz-sim-imu-system" name="gz::sim::systems::Imu"/>
+    </gazebo>
+  </xacro:macro>
 </robot>
