Commit message: thermal camera working

File: 41068_ignition_bringup/urdf/husky.gazebo.xacro (robot description, xacro)
@@ -170,3 +170,32 @@
     </sensor>
   </gazebo>
+<gazebo reference="thermal_link">
+  <sensor name="thermal_cam" type="thermal_camera">
+    <always_on>true</always_on>
+    <update_rate>30</update_rate>
+    <visualize>true</visualize>
+    <topic>/model/husky/thermal/image</topic>
+    <gz_frame_id>thermal_link</gz_frame_id>
+    <camera>
+      <horizontal_fov>1.3963</horizontal_fov>
+      <image>
+        <width>320</width>
+        <height>240</height>
+        <format>L8</format>
+      </image>
+      <clip>
+        <near>0.1</near>
+        <far>40</far>
+      </clip>
+    </camera>
+    <!-- Thermal plugin: set temperature range the sensor maps to 0–255 -->
+    <plugin
+      filename="ignition-gazebo-thermal-sensor-system"
+      name="ignition::gazebo::systems::ThermalSensor">
+      <min_temp>300</min_temp>  <!-- 0 °C -->
+      <max_temp>700</max_temp>  <!-- 100 °C -->
+      <resolution>0.1</resolution>
+    </plugin>
+  </sensor>
+</gazebo>
 </robot>

File: 41068_ignition_bringup/urdf/husky.urdf.xacro (robot description, xacro)
@@ -165,3 +165,20 @@
   </joint>
   <link name="camera_depth_optical_frame"/>
+<link name="thermal_link">
+  <visual>
+    <geometry>
+      <box>
+        <size>0.05 0.05 0.05</size>
+      </box>
+    </geometry>
+    <material>
+      <color rgba="0 0 1 1"/>
+    </material>
+  </visual>
+</link>
+<joint name="thermal_joint" type="fixed">
+  <parent link="base_link"/>
+  <child link="thermal_link"/>
+  <origin xyz="0.2 0 0.3" rpy="0 0 0"/>
+</joint>
 </robot>

Commit message: merged sensors branch to main

File: 41068_ignition_bringup/urdf/husky.gazebo.xacro (robot description, xacro)
@@ -199,49 +199,3 @@
   </sensor>
 </gazebo>
-  <!-- Thermal camera mounted on camera_link -->
-  <gazebo reference="thermal_link">
-    <sensor name="thermal_cam" type="thermal_camera">
-      <always_on>true</always_on>
-      <update_rate>5</update_rate>
-      <visualize>false</visualize>
-      <topic>/model/husky/thermal/image</topic>
-      <gz_frame_id>thermal_link</gz_frame_id>
-      <camera>
-        <horizontal_fov>1.3963</horizontal_fov>
-        <image>
-          <width>320</width>
-          <height>240</height>
-          <format>L8</format>
-        </image>
-        <clip>
-          <near>0.1</near>
-          <far>40</far>
-        </clip>
-      </camera>
-    </sensor>
-  </gazebo>
-<gazebo>
-    <plugin
-      filename="ignition-gazebo-logicalaudiosensorplugin-system"
-      name="gz::sim::systems::LogicalAudioSensorPlugin">
-      <!-- Microphone mounted at the robot base (pose is in model frame) -->
-      <microphone>
-        <id>1</id>
-        <pose>0 0 0 0 0 0</pose>
-        <volume_threshold>0.3</volume_threshold>
-      </microphone>
-      <!-- Optional beacon on the robot for testing; remove if you only want a mic -->
-      <source>
-        <id>1</id>
-        <pose>0.3 0 0.7 0 0 0</pose>
-        <attenuation_function>linear</attenuation_function>
-        <attenuation_shape>sphere</attenuation_shape>
-        <inner_radius>1.0</inner_radius>
-        <falloff_distance>6.0</falloff_distance>
-        <volume_level>0.5</volume_level>
-        <playing>true</playing>        <!-- start/stop at runtime -->
-        <play_duration>0</play_duration> <!-- 0 = infinite when playing -->
-      </source>
-    </plugin>
-  </gazebo>
 </robot>

File: 41068_ignition_bringup/urdf/husky.urdf.xacro (robot description, xacro)
@@ -165,20 +165,20 @@
   </joint>
   <link name="camera_depth_optical_frame"/>
-<link name="thermal_link">
-  <visual>
-    <geometry>
-      <box>
-        <size>0.05 0.05 0.05</size>
-      </box>
-    </geometry>
-    <material>
-      <color rgba="0 0 1 1"/>
-    </material>
-  </visual>
-</link>
-<joint name="thermal_joint" type="fixed">
-  <parent link="base_link"/>
-  <child link="thermal_link"/>
-  <origin xyz="0.2 0 0.3" rpy="0 0 0"/>
-</joint>
+  <link name="thermal_link">
+    <visual>
+      <geometry>
+        <box>
+          <size>0.05 0.05 0.05</size>
+        </box>
+      </geometry>
+      <material>
+        <color rgba="0 0 1 1"/>
+      </material>
+    </visual>
+  </link>
+  <joint name="thermal_joint" type="fixed">
+    <parent link="base_link"/>
+    <child link="thermal_link"/>
+    <origin xyz="0.2 0 0.3" rpy="0 0 0"/>
+  </joint>
 </robot>
