Commit message: New world. Disabled thermal

File: 41068_ignition_bringup/urdf/husky.urdf.xacro (robot description, xacro)
@@ -165,5 +165,5 @@
   </joint>
   <link name="camera_depth_optical_frame"/>
-  <link name="thermal_link">
+  <!-- <link name="thermal_link">
     <visual>
       <geometry>
@@ -181,4 +181,4 @@
     <child link="thermal_link"/>
     <origin xyz="0.2 0 0.3" rpy="0 0 0"/>
-  </joint>
+  </joint> -->
 </robot>

Commit message: Enabled thermal camera

File: 41068_ignition_bringup/urdf/husky.urdf.xacro (robot description, xacro)
@@ -165,5 +165,5 @@
   </joint>
   <link name="camera_depth_optical_frame"/>
-  <!-- <link name="thermal_link">
+  <link name="thermal_link">
     <visual>
       <geometry>
@@ -181,4 +181,4 @@
     <child link="thermal_link"/>
     <origin xyz="0.2 0 0.3" rpy="0 0 0"/>
-  </joint> -->
+  </joint>
 </robot>
