Commit message: Fixed RGB Camera

File: go2_description/xacro/gazebo_v2.xacro (robot description, xacro)
@@ -125,5 +125,5 @@
       <range>
         <min>0.05</min>
-        <max>12</max>
+        <max>24</max>
         <resolution>0.01</resolution>
       </range>
@@ -137,27 +137,33 @@
 </gazebo>
     <!-- CAMERA -->
-    <gazebo reference="camera_face">
-      <sensor name="camera" type="camera">
-        <pose>0 0 0 0 0 0</pose>
-        <visualize>true</visualize>
-        <update_rate>10</update_rate>
-        <camera>
-          <camera_info_topic>model/${robot_name}/color/camera_info</camera_info_topic>
-          <horizontal_fov>1.089</horizontal_fov>
-          <image>
-            <format>R8G8B8</format>
-            <width>640</width>
-            <height>480</height>
-          </image>
-          <clip>
-            <near>0.05</near>
-            <far>8.0</far>
-          </clip>
-        </camera>
-        <topic>model/${robot_name}/color/image_raw</topic>
-        <gz_frame_id>camera_face</gz_frame_id>
-      </sensor>
-    </gazebo>
-    <!-- ✅ ODOMETRY -->
+    <!-- RGB camera sensor -->
+<gazebo reference="camera_link">
+  <sensor name="rgbd_camera" type="rgbd_camera">
+    <camera>
+      <horizontal_fov>1.5</horizontal_fov> <!-- can adjust -->
+      <image>
+        <width>640</width>
+        <height>480</height>
+        <format>R8G8B8</format>
+      </image>
+      <clip>
+        <near>0.05</near>
+        <far>10</far>
+      </clip>
+      <depth_camera>
+        <clip>
+          <near>0.05</near>
+          <far>10</far>
+        </clip>
+      </depth_camera>
+    </camera>
+    <always_on>1</always_on>
+    <update_rate>10</update_rate>
+    <visualize>true</visualize>
+    <topic>/model/${robot_name}/camera</topic>
+    <gz_frame_id>camera_link</gz_frame_id>
+  </sensor>
+</gazebo>
+    <!-- ✅ ODOMETRY
     <gazebo>
       <plugin filename="ignition-gazebo-odometry-publisher-system"
@@ -168,5 +174,5 @@
         <robot_base_frame>base_link</robot_base_frame>
       </plugin>
-    </gazebo>
+    </gazebo> -->
     <!-- ✅ CMD_VEL VELOCITY CONTROL -->
     <!-- <gazebo>

File: go2_description/xacro/robot.xacro (robot description, xacro)
@@ -157,29 +157,45 @@
     </link>
   -->
-    <joint name="camera_face_joint" type="fixed">
-        <parent link="base_link"/>
-        <child link="camera_face"/>
-        <origin xyz="0.33 0 0.0057" rpy="0 0 0"/>
-    </joint>
-    <link name="camera_face">
-        <inertial>
-            <mass value="0.001"/>
-            <origin rpy="0 0 0" xyz="0 0 0"/>
-            <inertia ixx="0.0001" ixy="0" ixz="0" iyy="0.0001" iyz="0" izz="0.0001"/>
-        </inertial>
-        <visual>
-            <origin rpy="0 0 0" xyz="0 0 0"/>
-            <geometry>
-                <box size="0.001 0.001 0.001"/>
-            </geometry>
-            <!-- <material name="red"/> -->
-        </visual>
-        <collision>
-            <origin rpy="0 0 0" xyz="0 0 0"/>
-            <geometry>
-                <box size="0.001 0.001 0.001"/>
-            </geometry>
-        </collision>
-    </link>
+    <!-- Camera mount joint (relative to base_link) -->
+    <joint name="camera_joint" type="fixed">
+    <origin xyz="0.33 0.0 0.05" rpy="0 0 0"/>  <!-- adjust forward & height -->
+    <parent link="base_link"/>
+    <child link="camera_link"/>
+    </joint>
+    <link name="camera_link">
+    <visual>
+        <origin xyz="0 0 0" rpy="0 0 0"/>
+        <geometry>
+        <box size="0.02 0.08 0.05"/>
+        </geometry>
+        <material name="dark"/>
+    </visual>
+    </link>
+    <!-- ================= RGB CAMERA ================= -->
+    <joint name="camera_rgb_joint" type="fixed">
+    <origin xyz="0.005 0.018 0.013" rpy="0 0 0"/> <!-- offsets similar to Husky -->
+    <parent link="camera_link"/>
+    <child link="camera_rgb_frame"/>
+    </joint>
+    <link name="camera_rgb_frame"/>
+    <joint name="camera_rgb_optical_joint" type="fixed">
+    <origin xyz="0 0 0" rpy="-1.57 0 -1.57"/>
+    <parent link="camera_rgb_frame"/>
+    <child link="camera_rgb_optical_frame"/>
+    </joint>
+    <link name="camera_rgb_optical_frame"/>
+    <!-- ================= DEPTH CAMERA ================= -->
+    <joint name="camera_depth_joint" type="fixed">
+    <origin xyz="0.005 0.028 0.013" rpy="0 0 0"/> <!-- offset by depth_offset -->
+    <parent link="camera_link"/>
+    <child link="camera_depth_frame"/>
+    </joint>
+    <link name="camera_depth_frame"/>
+    <joint name="camera_depth_optical_joint" type="fixed">
+    <origin xyz="0 0 0" rpy="-1.57 0 -1.57"/>
+    <parent link="camera_depth_frame"/>
+    <child link="camera_depth_optical_frame"/>
+    </joint>
+    <link name="camera_depth_optical_frame"/>
     <xacro:leg name="rf" mirror="-1" mirror_dae= "False" front_hind="1"  front_hind_dae="True"  />
     <xacro:leg name="lf" mirror="1"  mirror_dae="True"   front_hind="1"  front_hind_dae="True"  />

Commit message: Robot Dog has all functionality which is similar with husky now

File: go2_description/xacro/gazebo_v2.xacro (robot description, xacro)
@@ -165,4 +165,33 @@
   </sensor>
 </gazebo>
+  <!-- ================= THERMAL CAMERA SENSOR ================= -->
+  <gazebo reference="thermal_link">
+    <sensor name="thermal_cam" type="thermal_camera">
+      <always_on>true</always_on>
+      <update_rate>5</update_rate>
+      <visualize>true</visualize>
+      <topic>/model/${robot_name}/thermal/image</topic>
+      <gz_frame_id>thermal_link</gz_frame_id>
+      <camera>
+        <horizontal_fov>1.3963</horizontal_fov> <!-- ~80 degrees -->
+        <image>
+          <width>320</width>
+          <height>240</height>
+          <format>L16</format>
+        </image>
+        <clip>
+          <near>0.1</near>
+          <far>40</far>
+        </clip>
+      </camera>
+      <plugin
+        filename="ignition-gazebo-thermal-sensor-system"
+        name="ignition::gazebo::systems::ThermalSensor">
+        <min_temp>300</min_temp>  <!-- 0 °C -->
+        <max_temp>700</max_temp>  <!-- 100 °C -->
+        <resolution>0.1</resolution>
+      </plugin>
+    </sensor>
+  </gazebo>
     <!-- ✅ ODOMETRY
     <gazebo>

File: go2_description/xacro/robot.xacro (robot description, xacro)
@@ -164,11 +164,11 @@
     </joint>
     <link name="camera_link">
-    <visual>
+    <!-- <visual>
         <origin xyz="0 0 0" rpy="0 0 0"/>
         <geometry>
-        <box size="0.02 0.08 0.05"/>
+        <box size="0.01 0.01 0.01"/>
         </geometry>
         <material name="dark"/>
-    </visual>
+    </visual> -->
     </link>
     <!-- ================= RGB CAMERA ================= -->
@@ -198,4 +198,12 @@
     </joint>
     <link name="camera_depth_optical_frame"/>
+      <!-- ================= THERMAL CAMERA ================= -->
+  <joint name="thermal_joint" type="fixed">
+    <origin xyz="0.33 0.0 0.03" rpy="0 0 0"/> <!-- Adjust position -->
+    <parent link="base_link"/>
+    <child link="thermal_link"/>
+  </joint>
+  <link name="thermal_link">
+  </link>
     <xacro:leg name="rf" mirror="-1" mirror_dae= "False" front_hind="1"  front_hind_dae="True"  />
     <xacro:leg name="lf" mirror="1"  mirror_dae="True"   front_hind="1"  front_hind_dae="True"  />

Commit message: Done localization for human, need to work with icon in rviz map based on the calculated pose

File: go2_description/xacro/gazebo_v2.xacro (robot description, xacro)
@@ -163,5 +163,5 @@
     <topic>/model/${robot_name}/camera</topic>
     <camera_info_topic>/model/${robot_name}/camera/camera_info</camera_info_topic>
-    <gz_frame_id>camera_link</gz_frame_id>
+    <gz_frame_id>camera_depth_optical_frame</gz_frame_id>
   </sensor>
 </gazebo>
@@ -175,15 +175,15 @@
     <topic>/model/${robot_name}/thermal/image</topic>
     <camera_info_topic>/model/${robot_name}/thermal/camera_info</camera_info_topic>
-    <gz_frame_id>thermal_link</gz_frame_id>
+    <gz_frame_id>thermal_optical_frame</gz_frame_id>
     <camera>
-      <horizontal_fov>1.3963</horizontal_fov> <!-- ~80 degrees -->
+      <horizontal_fov>1.5</horizontal_fov>
       <image>
-        <width>320</width>
-        <height>240</height>
+        <width>640</width>
+        <height>480</height>
         <format>L16</format>
       </image>
       <clip>
-        <near>0.1</near>
-        <far>40</far>
+        <near>0.05</near>
+        <far>10</far>
       </clip>
     </camera>

File: go2_description/xacro/robot.xacro (robot description, xacro)
@@ -107,54 +107,5 @@
         </collision>
     </link>
-    <!-- <joint name="imu_joint" type="fixed">
-        <parent link="trunk"/>
-        <child link="imu_link"/>
-        <origin rpy="0 0 0" xyz="0 0 0"/>
-    </joint>
-    <link name="imu_link">
-        <inertial>
-            <mass value="0.001"/>
-            <origin rpy="0 0 0" xyz="0 0 0"/>
-            <inertia ixx="0.0001" ixy="0" ixz="0" iyy="0.0001" iyz="0" izz="0.0001"/>
-        </inertial>
-        <visual>
-            <origin rpy="0 0 0" xyz="0 0 0"/>
-            <geometry>
-                <box size="0.001 0.001 0.001"/>
-            </geometry>
-        </visual>
-        <collision>
-            <origin rpy="0 0 0" xyz="0 0 0"/>
-            <geometry>
-                <box size=".001 .001 .001"/>
-            </geometry>
-        </collision>
-    </link> -->
-    <!--
-    <joint name="load_joint" type="fixed">
-        <parent link="trunk"/>
-        <child link="load_link"/>
-        <origin rpy="0 0 0" xyz="0 0 0"/>
-    </joint>
-    <link name="load_link">
-        <inertial>
-            <mass value="5"/>
-            <origin rpy="0 0 0" xyz="0 0 0"/>
-            <inertia ixx="0.01" ixy="0" ixz="0" iyy="0.01" iyz="0" izz="0.01"/>
-        </inertial>
-        <visual>
-            <origin rpy="0 0 0" xyz="0 0 0.2"/>
-            <geometry>
-                <box size="0.5 0.3 0.2"/>
-            </geometry>
-        </visual>
-        <collision>
-            <origin rpy="0 0 0" xyz="0 0 0"/>
-            <geometry>
-                <box size=".001 .001 .001"/>
-            </geometry>
-        </collision>
-    </link>
-  -->
+    <!-- ================= CAMERA MOUNT ================= -->
     <!-- Camera mount joint (relative to base_link) -->
     <joint name="camera_joint" type="fixed">
@@ -174,5 +125,5 @@
     <!-- ================= RGB CAMERA ================= -->
     <joint name="camera_rgb_joint" type="fixed">
-    <origin xyz="0.005 0.018 0.013" rpy="0 0 0"/> <!-- offsets similar to Husky -->
+    <origin xyz="0.33 0.0 0.03" rpy="0 0 0"/> <!-- offsets similar to Husky -->
     <parent link="camera_link"/>
     <child link="camera_rgb_frame"/>
@@ -180,5 +131,5 @@
     <link name="camera_rgb_frame"/>
     <joint name="camera_rgb_optical_joint" type="fixed">
-    <origin xyz="0 0 0" rpy="-1.57 0 -1.57"/>
+    <origin xyz="0 0 0" rpy="0 0 0"/>
     <parent link="camera_rgb_frame"/>
     <child link="camera_rgb_optical_frame"/>
@@ -187,5 +138,5 @@
     <!-- ================= DEPTH CAMERA ================= -->
     <joint name="camera_depth_joint" type="fixed">
-    <origin xyz="0.005 0.028 0.013" rpy="0 0 0"/> <!-- offset by depth_offset -->
+    <origin xyz="0.33 0.0 0.03" rpy="0 0 0"/> <!-- offset by depth_offset -->
     <parent link="camera_link"/>
     <child link="camera_depth_frame"/>
@@ -193,5 +144,5 @@
     <link name="camera_depth_frame"/>
     <joint name="camera_depth_optical_joint" type="fixed">
-    <origin xyz="0 0 0" rpy="-1.57 0 -1.57"/>
+    <origin xyz="0 0 0" rpy="0 0 0"/>
     <parent link="camera_depth_frame"/>
     <child link="camera_depth_optical_frame"/>
@@ -199,11 +150,16 @@
     <link name="camera_depth_optical_frame"/>
       <!-- ================= THERMAL CAMERA ================= -->
-  <joint name="thermal_joint" type="fixed">
+    <joint name="thermal_joint" type="fixed">
     <origin xyz="0.33 0.0 0.03" rpy="0 0 0"/> <!-- Adjust position -->
-    <parent link="base_link"/>
+    <parent link="camera_link"/>
     <child link="thermal_link"/>
-  </joint>
-  <link name="thermal_link">
-  </link>
+    </joint>
+    <link name="thermal_link"/>
+    <joint name="thermal_optical_joint" type="fixed">
+    <origin xyz="0 0 0" rpy="0 0 0"/>
+    <parent link="thermal_link"/>
+    <child link="thermal_optical_frame"/>
+    </joint>
+    <link name="thermal_optical_frame"/>
     <xacro:leg name="rf" mirror="-1" mirror_dae= "False" front_hind="1"  front_hind_dae="True"  />
     <xacro:leg name="lf" mirror="1"  mirror_dae="True"   front_hind="1"  front_hind_dae="True"  />

Commit message: Thermal

File: go2_description/xacro/gazebo_v2.xacro (robot description, xacro)
@@ -141,5 +141,6 @@
   <sensor name="rgbd_camera" type="rgbd_camera">
     <camera>
-      <horizontal_fov>1.5</horizontal_fov> <!-- can adjust -->
+      <horizontal_fov>1.57</horizontal_fov> <!-- can adjust -->
+      <vertical_fov>1.57</vertical_fov>
       <image>
         <width>640</width>
@@ -158,6 +159,6 @@
       </depth_camera>
     </camera>
-    <always_on>1</always_on>
-    <update_rate>10</update_rate>
+    <always_on>true</always_on>
+    <update_rate>5</update_rate>
     <visualize>true</visualize>
     <topic>/model/${robot_name}/camera</topic>
@@ -177,5 +178,6 @@
     <gz_frame_id>thermal_optical_frame</gz_frame_id>
     <camera>
-      <horizontal_fov>1.5</horizontal_fov>
+      <horizontal_fov>1.57</horizontal_fov>
+      <vertical_fov>1.57</vertical_fov>
       <image>
         <width>640</width>

File: go2_description/xacro/robot.xacro (robot description, xacro)
@@ -110,20 +110,27 @@
     <!-- Camera mount joint (relative to base_link) -->
     <joint name="camera_joint" type="fixed">
-    <origin xyz="0.33 0.0 0.05" rpy="0 0 0"/>  <!-- adjust forward & height -->
+    <origin xyz="0.33 0.0 0.04" rpy="0 0 0"/>  <!-- adjust forward & height -->
     <parent link="base_link"/>
     <child link="camera_link"/>
     </joint>
     <link name="camera_link">
-    <!-- <visual>
+        <!-- <visual>
         <origin xyz="0 0 0" rpy="0 0 0"/>
         <geometry>
-        <box size="0.01 0.01 0.01"/>
+            <box size="0.02 0.08 0.05"/>
         </geometry>
         <material name="dark"/>
-    </visual> -->
+        </visual>
+        <visual>
+        <origin xyz="0.015 0 0" rpy="0 1.57 0"/>
+        <geometry>
+            <cylinder length="0.03" radius="0.02"/>
+        </geometry>
+        <material name="dark"/>
+        </visual> -->
     </link>
     <!-- ================= RGB CAMERA ================= -->
     <joint name="camera_rgb_joint" type="fixed">
-    <origin xyz="0.33 0.0 0.03" rpy="0 0 0"/> <!-- offsets similar to Husky -->
+    <origin xyz="0.005 0.018 0.013" rpy="0 0 0"/> <!-- offsets similar to Husky -->
     <parent link="camera_link"/>
     <child link="camera_rgb_frame"/>
@@ -138,5 +145,5 @@
     <!-- ================= DEPTH CAMERA ================= -->
     <joint name="camera_depth_joint" type="fixed">
-    <origin xyz="0.33 0.0 0.03" rpy="0 0 0"/> <!-- offset by depth_offset -->
+    <origin xyz="0.005 0.018 0.013" rpy="0 0 0"/> <!-- offset by depth_offset -->
     <parent link="camera_link"/>
     <child link="camera_depth_frame"/>
@@ -151,5 +158,5 @@
       <!-- ================= THERMAL CAMERA ================= -->
     <joint name="thermal_joint" type="fixed">
-    <origin xyz="0.33 0.0 0.03" rpy="0 0 0"/> <!-- Adjust position -->
+    <origin xyz="0.005 0.018 0.013" rpy="0 0 0"/> <!-- Adjust position -->
     <parent link="camera_link"/>
     <child link="thermal_link"/>
