Commit message: Improve the localization

File: go2_description/xacro/robot.xacro (robot description, xacro)
@@ -132,5 +132,5 @@
     <!-- ================= RGB CAMERA ================= -->
     <joint name="camera_rgb_joint" type="fixed">
-    <origin xyz="0.005 0.018 0.013" rpy="0 0 0"/> <!-- offsets similar to Husky -->
+    <origin xyz="0.005 0 0" rpy="0 0 0"/> <!-- offsets similar to Husky -->
     <parent link="camera_link"/>
     <child link="camera_rgb_frame"/>
@@ -138,5 +138,5 @@
     <link name="camera_rgb_frame"/>
     <joint name="camera_rgb_optical_joint" type="fixed">
-    <origin xyz="0 0 0" rpy="0 0 0"/>
+    <origin xyz="0 0 0" rpy="-1.57 0 -1.57"/>
     <parent link="camera_rgb_frame"/>
     <child link="camera_rgb_optical_frame"/>
@@ -145,5 +145,5 @@
     <!-- ================= DEPTH CAMERA ================= -->
     <joint name="camera_depth_joint" type="fixed">
-    <origin xyz="0.005 0.018 0.013" rpy="0 0 0"/> <!-- offset by depth_offset -->
+    <origin xyz="0.005 0 0" rpy="0 0 0"/> <!-- offset by depth_offset -->
     <parent link="camera_link"/>
     <child link="camera_depth_frame"/>
@@ -151,5 +151,5 @@
     <link name="camera_depth_frame"/>
     <joint name="camera_depth_optical_joint" type="fixed">
-    <origin xyz="0 0 0" rpy="0 0 0"/>
+    <origin xyz="0 0 0" rpy="-1.57 0 -1.57"/>
     <parent link="camera_depth_frame"/>
     <child link="camera_depth_optical_frame"/>
@@ -158,5 +158,5 @@
       <!-- ================= THERMAL CAMERA ================= -->
     <joint name="thermal_joint" type="fixed">
-    <origin xyz="0.005 0.018 0.013" rpy="0 0 0"/> <!-- Adjust position -->
+    <origin xyz="0.005 0 0" rpy="0 0 0"/> <!-- Adjust position -->
     <parent link="camera_link"/>
     <child link="thermal_link"/>
@@ -164,5 +164,5 @@
     <link name="thermal_link"/>
     <joint name="thermal_optical_joint" type="fixed">
-    <origin xyz="0 0 0" rpy="0 0 0"/>
+    <origin xyz="0 0 0" rpy="-1.57 0 -1.57"/>
     <parent link="thermal_link"/>
     <child link="thermal_optical_frame"/>
